Commit message: [unfinished] writing arm.xacro for the project's arm

File: catkin_ws/src/arm_description/urdf/arm.xacro (robot description, xacro)
@@ -4,9 +4,9 @@
   <!-- Constants for robot dimensions -->
   <xacro:property name="PI" value="3.1415926535897931"/>
-  <xacro:property name="width" value="0.1" /> <!-- Square dimensions (widthxwidth) of beams -->
+  <xacro:property name="width" value="0.5" /> <!-- Square dimensions (widthxwidth) of beams -->
   <xacro:property name="height1" value="2" /> <!-- Link 1 -->
-  <xacro:property name="height2" value="1" /> <!-- Link 2 -->
-  <xacro:property name="height3" value="1" /> <!-- Link 3 -->
-  <xacro:property name="camera_link" value="0.05" /> <!-- Size of square 'camera' box -->
+  <xacro:property name="height2" value="1.5" /> <!-- Link 2 -->
+  <xacro:property name="height3" value="0.5" /> <!-- Link 3 -->
+  <xacro:property name="elbow_width" value="0.6" /> <!-- The length of elbow -->
   <xacro:property name="axel_offset" value="0.05" /> <!-- Space btw top of beam and the each joint -->
   <!-- Import all Gazebo-customization elements, including Gazebo colors -->
@@ -44,28 +44,28 @@
     </inertial>
   </link>
-  <joint name="joint1" type="continuous">
+  <joint name="elbow1_1" type="continuous">
     <parent link="link1"/>
-    <child link="link2"/>
-    <origin xyz="0 ${width} ${height1 - axel_offset}" rpy="0 0 0"/>
-    <axis xyz="0 1 0"/>
+    <child link="elbow1"/>
+    <origin xyz="0 0 ${height1}" rpy="0 0 0"/>
+    <axis xyz="0 0 1"/>
     <dynamics damping="0.7"/>
   </joint>
-  <!-- Middle Link -->
-  <link name="link2">
+  <!-- Elbow Link -->
+  <link name="elbow1">
     <collision>
-      <origin xyz="0 0 ${height2/2 - axel_offset}" rpy="0 0 0"/>
+      <origin xyz="0 0 ${elbow_width/2}" rpy="0 0 0"/>
       <geometry>
-	<box size="${width} ${width} ${height2}"/>
+	<box size="${elbow_width} ${elbow_width} ${elbow_width}"/>
       </geometry>
     </collision>
     <visual>
-      <origin xyz="0 0 ${height2/2 - axel_offset}" rpy="0 0 0"/>
+      <origin xyz="0 0 ${elbow_width/2}" rpy="0 0 0"/>
       <geometry>
-	<box size="${width} ${width} ${height2}"/>
+	<box size="${elbow_width} ${elbow_width} ${elbow_width}"/>
       </geometry>
-      <material name="black"/>
+      <material name="orange"/>
     </visual>
     <inertial>
-      <origin xyz="0 0 ${height2/2 - axel_offset}" rpy="0 0 0"/>
+      <origin xyz="0 0 ${elbow_width/2}" rpy="0 0 0"/>
       <mass value="1"/>
       <inertia
@@ -75,28 +75,28 @@
     </inertial>
   </link>
-  <joint name="joint2" type="continuous">
-    <parent link="link2"/>
-    <child link="link3"/>
-    <origin xyz="0 ${width} ${height2 - axel_offset*2}" rpy="0 0 0"/>
+  <joint name="elbow1_2" type="continuous">
+    <parent link="elbow1"/>
+    <child link="link2"/>
+    <origin xyz="0 ${elbow_width/2} ${elbow_width/2}" rpy="0 0 0"/>
     <axis xyz="0 1 0"/>
     <dynamics damping="0.7"/>
   </joint>
-  <!-- Top Link -->
-  <link name="link3">
+  <!-- Middle Link -->
+  <link name="link2">
     <collision>
-      <origin xyz="0 0 ${height3/2 - axel_offset}" rpy="0 0 0"/>
+      <origin xyz="0 ${width/2} ${height2/2}" rpy="0 0 0"/>
       <geometry>
-	<box size="${width} ${width} ${height3}"/>
+	<box size="${width} ${width} ${height2}"/>
       </geometry>
     </collision>
     <visual>
-      <origin xyz="0 0 ${height3/2 - axel_offset}" rpy="0 0 0"/>
+      <origin xyz="0 ${ width/2} ${height2/2}" rpy="0 0 0"/>
       <geometry>
-	<box size="${width} ${width} ${height3}"/>
+	<box size="${width} ${width} ${height2}"/>
       </geometry>
-      <material name="orange"/>
+      <material name="black"/>
     </visual>
     <inertial>
-      <origin xyz="0 0 ${height3/2 - axel_offset}" rpy="0 0 0"/>
+      <origin xyz="0 ${ width/2} ${height2/2}" rpy="0 0 0"/>
       <mass value="1"/>
       <inertia
@@ -106,73 +106,20 @@
     </inertial>
   </link>
-  <joint name="hokuyo_joint" type="fixed">
-    <axis xyz="0 1 0" />
-    <origin xyz="0 0 ${height3 - axel_offset/2}" rpy="0 0 0"/>
-    <parent link="link3"/>
-    <child link="hokuyo_link"/>
-  </joint>
-  <!-- Hokuyo Laser -->
-  <link name="hokuyo_link">
-    <collision>
-      <origin xyz="0 0 0" rpy="0 0 0"/>
-      <geometry>
-	<box size="0.1 0.1 0.1"/>
-      </geometry>
-    </collision>
-    <visual>
-      <origin xyz="0 0 0" rpy="0 0 0"/>
-      <geometry>
-        <mesh filename="package://arm_description/meshes/hokuyo.dae"/>
-      </geometry>
-    </visual>
-    <inertial>
-      <mass value="1e-5" />
-      <origin xyz="0 0 0" rpy="0 0 0"/>
-      <inertia ixx="1e-6" ixy="0" ixz="0" iyy="1e-6" iyz="0" izz="1e-6" />
-    </inertial>
-  </link>
-  <joint name="camera_joint" type="fixed">
-    <axis xyz="0 1 0" />
-    <origin xyz="${camera_link} 0 ${height3 - axel_offset*2}" rpy="0 0 0"/>
-    <parent link="link3"/>
-    <child link="camera_link"/>
-  </joint>
-  <!-- Camera -->
-  <link name="camera_link">
-    <collision>
-      <origin xyz="0 0 0" rpy="0 0 0"/>
-      <geometry>
-	<box size="${camera_link} ${camera_link} ${camera_link}"/>
-      </geometry>
-    </collision>
-    <visual>
-      <origin xyz="0 0 0" rpy="0 0 0"/>
-      <geometry>
-	<box size="${camera_link} ${camera_link} ${camera_link}"/>
-      </geometry>
-      <material name="red"/>
-    </visual>
-    <inertial>
-      <mass value="1e-5" />
-      <origin xyz="0 0 0" rpy="0 0 0"/>
-      <inertia ixx="1e-6" ixy="0" ixz="0" iyy="1e-6" iyz="0" izz="1e-6" />
-    </inertial>
-  </link>
-  <transmission name="tran1">
+  <transmission name="tran_elbow1_1">
     <type>transmission_interface/SimpleTransmission</type>
-    <joint name="joint1">
+    <joint name="elbow1_1">
       <hardwareInterface>EffortJointInterface</hardwareInterface>
     </joint>
-    <actuator name="motor1">
+    <actuator name="motor1_1">
       <hardwareInterface>EffortJointInterface</hardwareInterface>
       <mechanicalReduction>1</mechanicalReduction>
     </actuator>
   </transmission>
-  <transmission name="tran2">
+  <transmission name="tran_elbow1_2">
     <type>transmission_interface/SimpleTransmission</type>
-    <joint name="joint2">
+    <joint name="elbow1_2">
       <hardwareInterface>EffortJointInterface</hardwareInterface>
     </joint>
-    <actuator name="motor2">
+    <actuator name="motor1_2">
       <hardwareInterface>EffortJointInterface</hardwareInterface>
       <mechanicalReduction>1</mechanicalReduction>

Commit message: [finished] simple model with a torso(fixed,unmovable) and 3 links, joined to each other. Can run simulation and control by publishing rostopics.

File: catkin_ws/src/arm_description/urdf/arm.xacro (robot description, xacro)
@@ -5,5 +5,5 @@
   <xacro:property name="PI" value="3.1415926535897931"/>
   <xacro:property name="width" value="0.5" /> <!-- Square dimensions (widthxwidth) of beams -->
-  <xacro:property name="height1" value="2" /> <!-- Link 1 -->
+  <xacro:property name="height1" value="4" /> <!-- Link 1 -->
   <xacro:property name="height2" value="1.5" /> <!-- Link 2 -->
   <xacro:property name="height3" value="0.5" /> <!-- Link 3 -->
@@ -47,25 +47,25 @@
     <parent link="link1"/>
     <child link="elbow1"/>
-    <origin xyz="0 0 ${height1}" rpy="0 0 0"/>
-    <axis xyz="0 0 1"/>
-    <dynamics damping="0.7"/>
-  </joint>
-  <!-- Elbow Link -->
+    <origin xyz="0 ${width/2} ${height1-elbow_width/2}" rpy="0 0 0"/>
+    <axis xyz="0 1 0"/>
+    <dynamics damping="0.7"/>
+  </joint>
+  <!-- Elbow 1 Link -->
   <link name="elbow1">
     <collision>
-      <origin xyz="0 0 ${elbow_width/2}" rpy="0 0 0"/>
-      <geometry>
-	<box size="${elbow_width} ${elbow_width} ${elbow_width}"/>
-      </geometry>
-    </collision>
-    <visual>
-      <origin xyz="0 0 ${elbow_width/2}" rpy="0 0 0"/>
-      <geometry>
-	<box size="${elbow_width} ${elbow_width} ${elbow_width}"/>
-      </geometry>
-      <material name="orange"/>
-    </visual>
-    <inertial>
-      <origin xyz="0 0 ${elbow_width/2}" rpy="0 0 0"/>
+      <origin xyz="0 ${elbow_width/2} 0" rpy="0 0 0"/>
+      <geometry>
+	<box size="${elbow_width} ${elbow_width} ${elbow_width}"/>
+      </geometry>
+    </collision>
+    <visual>
+      <origin xyz="0 ${elbow_width/2} 0" rpy="0 0 0"/>
+      <geometry>
+	<box size="${elbow_width} ${elbow_width} ${elbow_width}"/>
+      </geometry>
+      <material name="orange"/>
+    </visual>
+    <inertial>
+      <origin xyz="0 ${elbow_width/2} 0" rpy="0 0 0"/>
       <mass value="1"/>
       <inertia
@@ -78,6 +78,6 @@
     <parent link="elbow1"/>
     <child link="link2"/>
-    <origin xyz="0 ${elbow_width/2} ${elbow_width/2}" rpy="0 0 0"/>
-    <axis xyz="0 1 0"/>
+    <origin xyz="0 ${elbow_width/2} ${-elbow_width/2}" rpy="0 0 0"/>
+    <axis xyz="1 0 0"/>
     <dynamics damping="0.7"/>
   </joint>
@@ -85,5 +85,5 @@
   <link name="link2">
     <collision>
-      <origin xyz="0 ${width/2} ${height2/2}" rpy="0 0 0"/>
+      <origin xyz="0 0 ${-height2/2}" rpy="0 0 0"/>
       <geometry>
 	<box size="${width} ${width} ${height2}"/>
@@ -91,5 +91,5 @@
     </collision>
     <visual>
-      <origin xyz="0 ${ width/2} ${height2/2}" rpy="0 0 0"/>
+      <origin xyz="0 0 ${-height2/2}" rpy="0 0 0"/>
       <geometry>
 	<box size="${width} ${width} ${height2}"/>
@@ -98,5 +98,98 @@
     </visual>
     <inertial>
-      <origin xyz="0 ${ width/2} ${height2/2}" rpy="0 0 0"/>
+      <origin xyz="0 0 ${-height2/2}" rpy="0 0 0"/>
+      <mass value="1"/>
+      <inertia
+	  ixx="1.0" ixy="0.0" ixz="0.0"
+	  iyy="1.0" iyz="0.0"
+	  izz="1.0"/>
+    </inertial>
+  </link>
+  <joint name="elbow2_1" type="continuous">
+    <parent link="link2"/>
+    <child link="elbow2"/>
+    <origin xyz="0 0 ${-height2}" rpy="0 0 0"/>
+    <axis xyz="0 0 1"/>
+    <dynamics damping="0.7"/>
+  </joint>
+  <!-- Elbow 2 Link -->
+  <link name="elbow2">
+    <collision>
+      <origin xyz="0 0 ${-elbow_width/2}" rpy="0 0 0"/>
+      <geometry>
+	<box size="${elbow_width} ${elbow_width} ${elbow_width}"/>
+      </geometry>
+    </collision>
+    <visual>
+      <origin xyz="0 0 ${-elbow_width/2}" rpy="0 0 0"/>
+      <geometry>
+	<box size="${elbow_width} ${elbow_width} ${elbow_width}"/>
+      </geometry>
+      <material name="orange"/>
+    </visual>
+    <inertial>
+      <origin xyz="0 0 ${-elbow_width/2}" rpy="0 0 0"/>
+      <mass value="1"/>
+      <inertia
+	  ixx="1.0" ixy="0.0" ixz="0.0"
+	  iyy="1.0" iyz="0.0"
+	  izz="1.0"/>
+    </inertial>
+  </link>
+  <joint name="elbow2_2" type="continuous">
+    <parent link="elbow2"/>
+    <child link="link3"/>
+    <origin xyz="0 0 ${-elbow_width}" rpy="0 0 0"/>
+    <axis xyz="1 0 0"/>
+    <dynamics damping="0.7"/>
+  </joint>
+  <!-- Palm Link -->
+  <link name="link3">
+    <collision>
+      <origin xyz="0 0 ${-height3/2}" rpy="0 0 0"/>
+      <geometry>
+	<box size="${width} ${width} ${height3}"/>
+      </geometry>
+    </collision>
+    <visual>
+      <origin xyz="0 0 ${-height3/2}" rpy="0 0 0"/>
+      <geometry>
+	<box size="${width} ${width} ${height3}"/>
+      </geometry>
+      <material name="black"/>
+    </visual>
+    <inertial>
+      <origin xyz="0 0 ${-height3/2}" rpy="0 0 0"/>
+      <mass value="1"/>
+      <inertia
+	  ixx="1.0" ixy="0.0" ixz="0.0"
+	  iyy="1.0" iyz="0.0"
+	  izz="1.0"/>
+    </inertial>
+  </link>
+  <joint name="elbow3_1" type="continuous">
+    <parent link="link3"/>
+    <child link="elbow3"/>
+    <origin xyz="0 0 ${-height3}" rpy="0 0 0"/>
+    <axis xyz="0 0 1"/>
+    <dynamics damping="0.7"/>
+  </joint>
+  <!-- Elbow 3 Link -->
+  <link name="elbow3">
+    <collision>
+      <origin xyz="0 0 ${-elbow_width/2}" rpy="0 0 0"/>
+      <geometry>
+	<box size="${elbow_width} ${elbow_width} ${elbow_width}"/>
+      </geometry>
+    </collision>
+    <visual>
+      <origin xyz="0 0 ${-elbow_width/2}" rpy="0 0 0"/>
+      <geometry>
+	<box size="${elbow_width} ${elbow_width} ${elbow_width}"/>
+      </geometry>
+      <material name="orange"/>
+    </visual>
+    <inertial>
+      <origin xyz="0 0 ${-elbow_width/2}" rpy="0 0 0"/>
       <mass value="1"/>
       <inertia
@@ -126,3 +219,33 @@
     </actuator>
   </transmission>
+  <transmission name="tran_elbow2_1">
+    <type>transmission_interface/SimpleTransmission</type>
+    <joint name="elbow2_1">
+      <hardwareInterface>EffortJointInterface</hardwareInterface>
+    </joint>
+    <actuator name="motor2_1">
+      <hardwareInterface>EffortJointInterface</hardwareInterface>
+      <mechanicalReduction>1</mechanicalReduction>
+    </actuator>
+  </transmission>
+  <transmission name="tran_elbow2_2">
+    <type>transmission_interface/SimpleTransmission</type>
+    <joint name="elbow2_2">
+      <hardwareInterface>EffortJointInterface</hardwareInterface>
+    </joint>
+    <actuator name="motor2_2">
+      <hardwareInterface>EffortJointInterface</hardwareInterface>
+      <mechanicalReduction>1</mechanicalReduction>
+    </actuator>
+  </transmission>
+  <transmission name="tran_elbow3_1">
+    <type>transmission_interface/SimpleTransmission</type>
+    <joint name="elbow3_1">
+      <hardwareInterface>EffortJointInterface</hardwareInterface>
+    </joint>
+    <actuator name="motor3_1">
+      <hardwareInterface>EffortJointInterface</hardwareInterface>
+      <mechanicalReduction>1</mechanicalReduction>
+    </actuator>
+  </transmission>
 </robot>

Commit message: nothing much, editted xacro file and changed folder structer

File: catkin_ws/src/arm_description/urdf/arm.xacro (robot description, xacro)
@@ -8,5 +8,5 @@
   <xacro:property name="height2" value="1.5" /> <!-- Link 2 -->
   <xacro:property name="height3" value="0.5" /> <!-- Link 3 -->
-  <xacro:property name="elbow_width" value="0.6" /> <!-- The length of elbow -->
+  <xacro:property name="elbow_width" value="0.1" /> <!-- The length of elbow -->
   <xacro:property name="axel_offset" value="0.05" /> <!-- Space btw top of beam and the each joint -->
   <!-- Import all Gazebo-customization elements, including Gazebo colors -->

Commit message: added stl meshes: 1 dummy body, joints, changing initial viewpoint of arm.world

File: catkin_ws/src/arm_description/urdf/arm.xacro (robot description, xacro)
@@ -4,9 +4,9 @@
   <!-- Constants for robot dimensions -->
   <xacro:property name="PI" value="3.1415926535897931"/>
-  <xacro:property name="width" value="0.5" /> <!-- Square dimensions (widthxwidth) of beams -->
-  <xacro:property name="height1" value="4" /> <!-- Link 1 -->
-  <xacro:property name="height2" value="1.5" /> <!-- Link 2 -->
-  <xacro:property name="height3" value="0.5" /> <!-- Link 3 -->
-  <xacro:property name="elbow_width" value="0.1" /> <!-- The length of elbow -->
+  <xacro:property name="width" value="1.0" /> <!-- Square dimensions (widthxwidth) of beams -->
+  <xacro:property name="height1" value="9" /> <!-- Link 1 -->
+  <xacro:property name="height2" value="2" /> <!-- Link 2 -->
+  <xacro:property name="height3" value="2" /> <!-- Link 3 -->
+  <xacro:property name="elbow_width" value="1.0" /> <!-- The length of elbow -->
   <xacro:property name="axel_offset" value="0.05" /> <!-- Space btw top of beam and the each joint -->
   <!-- Import all Gazebo-customization elements, including Gazebo colors -->
@@ -29,7 +29,8 @@
     </collision>
     <visual>
-      <origin xyz="0 0 ${height1/2}" rpy="0 0 0"/>
-      <geometry>
-	<box size="${width} ${width} ${height1}"/>
+      <origin xyz="${width*2.5} 0.5 0" rpy="1.57 0 -1.57"/>
+      <geometry>
+	<mesh filename="package://arm_description/meshes/dummyBody.STL" scale="2.7 2.7 2.7"/>
+	<!--box size="${width} ${width} ${height1}"/-->
       </geometry>
       <material name="orange"/>
@@ -60,7 +61,8 @@
     </collision>
     <visual>
-      <origin xyz="0 ${elbow_width/2} 0" rpy="0 0 0"/>
-      <geometry>
-	<box size="${elbow_width} ${elbow_width} ${elbow_width}"/>
+      <origin xyz="0 0 0" rpy="-1.57 1.57 0"/>
+      <geometry>
+	<mesh filename="package://arm_description/meshes/gearBox.STL" scale="0.2 0.2 0.2"/>
+	<!--box size="${elbow_width} ${elbow_width} ${elbow_width}"/-->
       </geometry>
       <material name="orange"/>
@@ -122,7 +124,7 @@
     </collision>
     <visual>
-      <origin xyz="0 0 ${-elbow_width/2}" rpy="0 0 0"/>
-      <geometry>
-	<box size="${elbow_width} ${elbow_width} ${elbow_width}"/>
+      <origin xyz="0 ${-elbow_width/1.3} 0" rpy="0 3.14 0"/>
+      <geometry>
+	<mesh filename="package://arm_description/meshes/gearBox.STL" scale="0.2 0.2 0.2"/>
       </geometry>
       <material name="orange"/>
@@ -184,7 +186,7 @@
     </collision>
     <visual>
-      <origin xyz="0 0 ${-elbow_width/2}" rpy="0 0 0"/>
-      <geometry>
-	<box size="${elbow_width} ${elbow_width} ${elbow_width}"/>
+      <origin xyz="0 0 0" rpy="-1.57 1.57 0"/>
+      <geometry>
+	<mesh filename="package://arm_description/meshes/gearBox.STL" scale="0.2 0.2 0.2"/>
       </geometry>
       <material name="orange"/>

Commit message: successfully assembled dummy body, shoulder joint and the first link.

File: catkin_ws/src/arm_description/urdf/arm.xacro (robot description, xacro)
@@ -29,7 +29,7 @@
     </collision>
     <visual>
-      <origin xyz="${width*2.5} 0.5 0" rpy="1.57 0 -1.57"/>
-      <geometry>
-	<mesh filename="package://arm_description/meshes/dummyBody.STL" scale="2.7 2.7 2.7"/>
+      <origin xyz="${width*2.0} 0.5 0" rpy="1.57 0 -1.57"/>
+      <geometry>
+	<mesh filename="package://arm_description/meshes/dummyBody.STL" scale="2 2.6 2"/>
 	<!--box size="${width} ${width} ${height1}"/-->
       </geometry>
@@ -61,5 +61,5 @@
     </collision>
     <visual>
-      <origin xyz="0 0 0" rpy="-1.57 1.57 0"/>
+      <origin xyz="${elbow_width/2.39} 0 ${elbow_width/2-0.13}" rpy="-1.57 1.57 0"/>
       <geometry>
 	<mesh filename="package://arm_description/meshes/gearBox.STL" scale="0.2 0.2 0.2"/>
@@ -80,5 +80,5 @@
     <parent link="elbow1"/>
     <child link="link2"/>
-    <origin xyz="0 ${elbow_width/2} ${-elbow_width/2}" rpy="0 0 0"/>
+    <origin xyz="0 ${elbow_width/2} ${-elbow_width*0}" rpy="0 0 0"/>
     <axis xyz="1 0 0"/>
     <dynamics damping="0.7"/>
@@ -93,7 +93,7 @@
     </collision>
     <visual>
-      <origin xyz="0 0 ${-height2/2}" rpy="0 0 0"/>
-      <geometry>
-	<box size="${width} ${width} ${height2}"/>
+      <origin xyz="${-width/2.3} 0 ${-height2/1}" rpy="1.57 0 0"/>
+      <geometry>
+	<mesh filename="package://arm_description/meshes/armSkeleton.STL" scale="0.2 0.26 0.2"/>
       </geometry>
       <material name="black"/>

Commit message: assembled Elbow joint (Elbow 2)

File: catkin_ws/src/arm_description/urdf/arm.xacro (robot description, xacro)
@@ -63,5 +63,5 @@
       <origin xyz="${elbow_width/2.39} 0 ${elbow_width/2-0.13}" rpy="-1.57 1.57 0"/>
       <geometry>
-	<mesh filename="package://arm_description/meshes/gearBox.STL" scale="0.2 0.2 0.2"/>
+	<mesh filename="package://arm_description/meshes/gearBox.STL" scale="0.2 0.2 0.25"/>
 	<!--box size="${elbow_width} ${elbow_width} ${elbow_width}"/-->
       </geometry>
@@ -93,5 +93,5 @@
     </collision>
     <visual>
-      <origin xyz="${-width/2.3} 0 ${-height2/1}" rpy="1.57 0 0"/>
+      <origin xyz="${-width/2.3} 0.1 ${-height2/1}" rpy="1.57 0 0"/>
       <geometry>
 	<mesh filename="package://arm_description/meshes/armSkeleton.STL" scale="0.2 0.26 0.2"/>
@@ -124,5 +124,5 @@
     </collision>
     <visual>
-      <origin xyz="0 ${-elbow_width/1.3} 0" rpy="0 3.14 0"/>
+      <origin xyz="${elbow_width/2.3} ${-elbow_width/2.35} 0.06" rpy="0 3.14 0"/>
       <geometry>
 	<mesh filename="package://arm_description/meshes/gearBox.STL" scale="0.2 0.2 0.2"/>

Commit message: assembled Link 2

File: catkin_ws/src/arm_description/urdf/arm.xacro (robot description, xacro)
@@ -124,5 +124,5 @@
     </collision>
     <visual>
-      <origin xyz="${elbow_width/2.3} ${-elbow_width/2.35} 0.06" rpy="0 3.14 0"/>
+      <origin xyz="${elbow_width/2.55} ${-elbow_width/2.45} 0.06" rpy="0 3.14 0"/>
       <geometry>
 	<mesh filename="package://arm_description/meshes/gearBox.STL" scale="0.2 0.2 0.2"/>
@@ -142,5 +142,5 @@
     <parent link="elbow2"/>
     <child link="link3"/>
-    <origin xyz="0 0 ${-elbow_width}" rpy="0 0 0"/>
+    <origin xyz="0 0 ${-elbow_width/3}" rpy="0 0 0"/>
     <axis xyz="1 0 0"/>
     <dynamics damping="0.7"/>
@@ -155,7 +155,7 @@
     </collision>
     <visual>
-      <origin xyz="0 0 ${-height3/2}" rpy="0 0 0"/>
-      <geometry>
-	<box size="${width} ${width} ${height3}"/>
+      <origin xyz="${-width/8.0} -0.47 ${-height2/1}" rpy="1.57 0 1.57"/>
+      <geometry>
+	<mesh filename="package://arm_description/meshes/armSkeleton.STL" scale="0.2 0.26 0.2"/>
       </geometry>
       <material name="black"/>

Commit message: assembled all

File: catkin_ws/src/arm_description/urdf/arm.xacro (robot description, xacro)
@@ -186,5 +186,5 @@
     </collision>
     <visual>
-      <origin xyz="0 0 0" rpy="-1.57 1.57 0"/>
+      <origin xyz="0.4 -0.4 0.05" rpy="0 3.14 0"/>
       <geometry>
 	<mesh filename="package://arm_description/meshes/gearBox.STL" scale="0.2 0.2 0.2"/>

Commit message: assembled all, can use topics to give commands. Basically done simulation for skeleton of one arm

File: catkin_ws/src/arm_description/urdf/arm.xacro (robot description, xacro)
@@ -40,7 +40,7 @@
       <mass value="1"/>
       <inertia
-	  ixx="3.0" ixy="0.0" ixz="0.0"
-	  iyy="3.0" iyz="0.0"
-	  izz="3.0"/>
+	  ixx="9.0" ixy="0.0" ixz="0.0"
+	  iyy="9.0" iyz="0.0"
+	  izz="9.0"/>
     </inertial>
   </link>
@@ -143,5 +143,5 @@
     <child link="link3"/>
     <origin xyz="0 0 ${-elbow_width/3}" rpy="0 0 0"/>
-    <axis xyz="1 0 0"/>
+    <axis xyz="0 1 0"/>
     <dynamics damping="0.7"/>
   </joint>
