Commit message: learning pr2 controller in pr2_* packages. Nothing new.

File: catkin_ws/src/arm_description/urdf/arm.xacro (robot description, xacro)
@@ -10,4 +10,8 @@
   <xacro:property name="elbow_width" value="1.0" /> <!-- The length of elbow -->
   <xacro:property name="axel_offset" value="0.05" /> <!-- Space btw top of beam and the each joint -->
+  <xacro:property name="limit_lower" value="-2" /> <!-- Space btw top of beam and the each joint -->
+  <xacro:property name="limit_upper" value="1" /> <!-- Space btw top of beam and the each joint -->
+  <xacro:property name="limit_effort" value="30" /> <!-- Space btw top of beam and the each joint -->
+  <xacro:property name="limit_velocity" value="30" /> <!-- Space btw top of beam and the each joint -->
   <!-- Import all Gazebo-customization elements, including Gazebo colors -->
   <xacro:include filename="$(find arm_description)/urdf/arm.gazebo" />
@@ -38,5 +42,5 @@
     <inertial>
       <origin xyz="0 0 ${height1/2}" rpy="0 0 0"/>
-      <mass value="1"/>
+      <mass value="10"/>
       <inertia
 	  ixx="9.0" ixy="0.0" ixz="0.0"
@@ -51,4 +55,6 @@
     <axis xyz="0 1 0"/>
     <dynamics damping="0.7"/>
+    <limit effort="${limit_effort}" lower="${limit_lower}" upper="${limit_upper}" velocity="${limit_velocity}" />
+    <safety_controller k_velocity="100" k_position="15" soft_lower_limit="-1.9" soft_upper_limit="0.5" />
   </joint>
   <!-- Elbow 1 Link -->
@@ -70,5 +76,5 @@
     <inertial>
       <origin xyz="0 ${elbow_width/2} 0" rpy="0 0 0"/>
-      <mass value="1"/>
+      <mass value="0.1"/>
       <inertia
 	  ixx="1.0" ixy="0.0" ixz="0.0"
@@ -101,5 +107,5 @@
     <inertial>
       <origin xyz="0 0 ${-height2/2}" rpy="0 0 0"/>
-      <mass value="1"/>
+      <mass value="0.1"/>
       <inertia
 	  ixx="1.0" ixy="0.0" ixz="0.0"
@@ -132,5 +138,5 @@
     <inertial>
       <origin xyz="0 0 ${-elbow_width/2}" rpy="0 0 0"/>
-      <mass value="1"/>
+      <mass value="0.1"/>
       <inertia
 	  ixx="1.0" ixy="0.0" ixz="0.0"
@@ -163,5 +169,5 @@
     <inertial>
       <origin xyz="0 0 ${-height3/2}" rpy="0 0 0"/>
-      <mass value="1"/>
+      <mass value="0.1"/>
       <inertia
 	  ixx="1.0" ixy="0.0" ixz="0.0"
@@ -194,5 +200,5 @@
     <inertial>
       <origin xyz="0 0 ${-elbow_width/2}" rpy="0 0 0"/>
-      <mass value="1"/>
+      <mass value="0.1"/>
       <inertia
 	  ixx="1.0" ixy="0.0" ixz="0.0"

Commit message: tuned PID for joints. Fast, but has (small) overshoot. Worked wuite realistic.

File: catkin_ws/src/arm_description/urdf/arm.xacro (robot description, xacro)
@@ -10,6 +10,6 @@
   <xacro:property name="elbow_width" value="1.0" /> <!-- The length of elbow -->
   <xacro:property name="axel_offset" value="0.05" /> <!-- Space btw top of beam and the each joint -->
-  <xacro:property name="limit_lower" value="-2" /> <!-- Space btw top of beam and the each joint -->
-  <xacro:property name="limit_upper" value="1" /> <!-- Space btw top of beam and the each joint -->
+  <xacro:property name="limit_lower" value="-1.57" /> <!-- Space btw top of beam and the each joint -->
+  <xacro:property name="limit_upper" value="1.57" /> <!-- Space btw top of beam and the each joint -->
   <xacro:property name="limit_effort" value="30" /> <!-- Space btw top of beam and the each joint -->
   <xacro:property name="limit_velocity" value="30" /> <!-- Space btw top of beam and the each joint -->
@@ -42,9 +42,9 @@
     <inertial>
       <origin xyz="0 0 ${height1/2}" rpy="0 0 0"/>
-      <mass value="10"/>
-      <inertia
-	  ixx="9.0" ixy="0.0" ixz="0.0"
-	  iyy="9.0" iyz="0.0"
-	  izz="9.0"/>
+      <mass value="1000"/>
+      <inertia
+	  ixx="190.0" ixy="0.0" ixz="0.0"
+	  iyy="190.0" iyz="0.0"
+	  izz="190.0"/>
     </inertial>
   </link>
@@ -78,7 +78,7 @@
       <mass value="0.1"/>
       <inertia
-	  ixx="1.0" ixy="0.0" ixz="0.0"
-	  iyy="1.0" iyz="0.0"
-	  izz="1.0"/>
+	  ixx="0.1" ixy="0.0" ixz="0.0"
+	  iyy="0.1" iyz="0.0"
+	  izz="0.1"/>
     </inertial>
   </link>
@@ -109,7 +109,7 @@
       <mass value="0.1"/>
       <inertia
-	  ixx="1.0" ixy="0.0" ixz="0.0"
-	  iyy="1.0" iyz="0.0"
-	  izz="1.0"/>
+	  ixx="10.1" ixy="0.0" ixz="0.0"
+	  iyy="10.1" iyz="0.0"
+	  izz="10.1"/>
     </inertial>
   </link>
@@ -120,4 +120,6 @@
     <axis xyz="0 0 1"/>
     <dynamics damping="0.7"/>
+    <limit effort="${limit_effort}" lower="${limit_lower}" upper="${limit_upper}" velocity="${limit_velocity}" />
+    <safety_controller k_velocity="100" k_position="15" soft_lower_limit="-1.9" soft_upper_limit="0.5" />
   </joint>
   <!-- Elbow 2 Link -->
@@ -140,7 +142,7 @@
       <mass value="0.1"/>
       <inertia
-	  ixx="1.0" ixy="0.0" ixz="0.0"
-	  iyy="1.0" iyz="0.0"
-	  izz="1.0"/>
+	  ixx="0.1" ixy="0.0" ixz="0.0"
+	  iyy="0.1" iyz="0.0"
+	  izz="0.1"/>
     </inertial>
   </link>
@@ -171,7 +173,7 @@
       <mass value="0.1"/>
       <inertia
-	  ixx="1.0" ixy="0.0" ixz="0.0"
-	  iyy="1.0" iyz="0.0"
-	  izz="1.0"/>
+	  ixx="3.1" ixy="0.0" ixz="0.0"
+	  iyy="3.1" iyz="0.0"
+	  izz="3.1"/>
     </inertial>
   </link>
@@ -202,7 +204,7 @@
       <mass value="0.1"/>
       <inertia
-	  ixx="1.0" ixy="0.0" ixz="0.0"
-	  iyy="1.0" iyz="0.0"
-	  izz="1.0"/>
+	  ixx="0.1" ixy="0.0" ixz="0.0"
+	  iyy="0.1" iyz="0.0"
+	  izz="0.1"/>
     </inertial>
   </link>

Commit message: new body

File: catkin_ws/src/arm_description/urdf/arm.xacro (robot description, xacro)
@@ -33,7 +33,7 @@
     </collision>
     <visual>
-      <origin xyz="${width*2.0} 0.5 0" rpy="1.57 0 -1.57"/>
-      <geometry>
-	<mesh filename="package://arm_description/meshes/dummyBody.STL" scale="2 2.6 2"/>
+      <origin xyz="${width*2} 0.5 0" rpy="1.57 0 -1.57"/>
+      <geometry>
+	<mesh filename="package://arm_description/meshes/square_body.STL" scale="3.55 3.55 3.55"/>
 	<!--box size="${width} ${width} ${height1}"/-->
       </geometry>

Commit message: dual arm, with body. Ready for demonstration in VGU Open day

File: catkin_ws/src/arm_description/urdf/arm.xacro (robot description, xacro)
@@ -5,5 +5,5 @@
   <xacro:property name="PI" value="3.1415926535897931"/>
   <xacro:property name="width" value="1.0" /> <!-- Square dimensions (widthxwidth) of beams -->
-  <xacro:property name="height1" value="9" /> <!-- Link 1 -->
+  <xacro:property name="height1" value="7.40" /> <!-- Link 1 -->
   <xacro:property name="height2" value="2" /> <!-- Link 2 -->
   <xacro:property name="height3" value="2" /> <!-- Link 3 -->
@@ -14,4 +14,9 @@
   <xacro:property name="limit_effort" value="30" /> <!-- Space btw top of beam and the each joint -->
   <xacro:property name="limit_velocity" value="30" /> <!-- Space btw top of beam and the each joint -->
+  <xacro:property name="scale" value="0.4" />
+  <xacro:property name="y_offset" value="0.14" />
+  <xacro:property name="x_offset" value="0.10" />
+  <xacro:property name="z_offset" value="0.10" />
+  <xacro:property name="leftArm_offset" value="2.5" />
   <!-- Import all Gazebo-customization elements, including Gazebo colors -->
   <xacro:include filename="$(find arm_description)/urdf/arm.gazebo" />
@@ -33,7 +38,7 @@
     </collision>
     <visual>
-      <origin xyz="${width*2} 0.5 0" rpy="1.57 0 -1.57"/>
-      <geometry>
-	<mesh filename="package://arm_description/meshes/square_body.STL" scale="3.55 3.55 3.55"/>
+      <origin xyz="1.1 -3.15 8" rpy="-1.57 0 1.57"/>
+      <geometry>
+	<mesh filename="package://arm_description/meshes/body.STL" scale="${scale+0.1} ${scale+0.1} ${scale+0.1}"/>
 	<!--box size="${width} ${width} ${height1}"/-->
       </geometry>
@@ -44,7 +49,7 @@
       <mass value="1000"/>
       <inertia
-	  ixx="190.0" ixy="0.0" ixz="0.0"
-	  iyy="190.0" iyz="0.0"
-	  izz="190.0"/>
+	  ixx="990.0" ixy="0.0" ixz="0.0"
+	  iyy="990.0" iyz="0.0"
+	  izz="990.0"/>
     </inertial>
   </link>
@@ -52,5 +57,5 @@
     <parent link="link1"/>
     <child link="elbow1"/>
-    <origin xyz="0 ${width/2} ${height1-elbow_width/2}" rpy="0 0 0"/>
+    <origin xyz="${x_offset} ${width/2} ${height1-elbow_width/2}" rpy="0 0 0"/>
     <axis xyz="0 1 0"/>
     <dynamics damping="0.7"/>
@@ -67,7 +72,7 @@
     </collision>
     <visual>
-      <origin xyz="${elbow_width/2.39} 0 ${elbow_width/2-0.13}" rpy="-1.57 1.57 0"/>
-      <geometry>
-	<mesh filename="package://arm_description/meshes/gearBox.STL" scale="0.2 0.2 0.25"/>
+      <origin xyz="${-elbow_width/2} 0 ${-elbow_width/2}" rpy="0 0 0"/>
+      <geometry>
+	<mesh filename="package://arm_description/meshes/shoulder_ball.STL" scale="0.4 0.4 0.4"/>
 	<!--box size="${elbow_width} ${elbow_width} ${elbow_width}"/-->
       </geometry>
@@ -86,5 +91,5 @@
     <parent link="elbow1"/>
     <child link="link2"/>
-    <origin xyz="0 ${elbow_width/2} ${-elbow_width*0}" rpy="0 0 0"/>
+    <origin xyz="0 ${elbow_width/2+0.04} ${-elbow_width*0}" rpy="0 0 0"/>
     <axis xyz="1 0 0"/>
     <dynamics damping="0.7"/>
@@ -99,9 +104,9 @@
     </collision>
     <visual>
-      <origin xyz="${-width/2.3} 0.1 ${-height2/1}" rpy="1.57 0 0"/>
-      <geometry>
-	<mesh filename="package://arm_description/meshes/armSkeleton.STL" scale="0.2 0.26 0.2"/>
-      </geometry>
-      <material name="black"/>
+      <origin xyz="${-elbow_width/2.7} ${-y_offset-0.4} ${height2/3.5}" rpy="-1.57 0 0"/>
+      <geometry>
+	<mesh filename="package://arm_description/meshes/shoulder_link.STL" scale="0.4 0.4 0.4"/>
+      </geometry>
+      <material name="orange"/>
     </visual>
     <inertial>
@@ -117,5 +122,5 @@
     <parent link="link2"/>
     <child link="elbow2"/>
-    <origin xyz="0 0 ${-height2}" rpy="0 0 0"/>
+    <origin xyz="0 0 ${-height2-z_offset}" rpy="0 0 0"/>
     <axis xyz="0 0 1"/>
     <dynamics damping="0.7"/>
@@ -132,7 +137,7 @@
     </collision>
     <visual>
-      <origin xyz="${elbow_width/2.55} ${-elbow_width/2.45} 0.06" rpy="0 3.14 0"/>
-      <geometry>
-	<mesh filename="package://arm_description/meshes/gearBox.STL" scale="0.2 0.2 0.2"/>
+      <origin xyz="${-elbow_width/2.5} ${-elbow_width/4-y_offset} ${z_offset-0.08}" rpy="-1.57 0 0"/>
+      <geometry>
+	<mesh filename="package://arm_description/meshes/elbow_ball.STL" scale="${scale} ${scale} ${scale}"/>
       </geometry>
       <material name="orange"/>
@@ -150,9 +155,9 @@
     <parent link="elbow2"/>
     <child link="link3"/>
-    <origin xyz="0 0 ${-elbow_width/3}" rpy="0 0 0"/>
-    <axis xyz="0 1 0"/>
-    <dynamics damping="0.7"/>
-  </joint>
-  <!-- Palm Link -->
+    <origin xyz="0 0 ${-elbow_width/2}" rpy="0 0 0"/>
+    <axis xyz="1 0 0"/>
+    <dynamics damping="0.7"/>
+  </joint>
+  <!-- Forearm Link -->
   <link name="link3">
     <collision>
@@ -163,7 +168,7 @@
     </collision>
     <visual>
-      <origin xyz="${-width/8.0} -0.47 ${-height2/1}" rpy="1.57 0 1.57"/>
-      <geometry>
-	<mesh filename="package://arm_description/meshes/armSkeleton.STL" scale="0.2 0.26 0.2"/>
+      <origin xyz="${-elbow_width/4.1} ${-elbow_width/4-y_offset} ${z_offset+0.3}" rpy="-1.57 0 0"/>
+      <geometry>
+	<mesh filename="package://arm_description/meshes/forearm_link.STL" scale="${scale} ${scale} ${scale}"/>
       </geometry>
       <material name="black"/>
@@ -181,6 +186,6 @@
     <parent link="link3"/>
     <child link="elbow3"/>
-    <origin xyz="0 0 ${-height3}" rpy="0 0 0"/>
-    <axis xyz="0 0 1"/>
+    <origin xyz="0 ${0.15-y_offset} ${-1.79+z_offset}" rpy="0 0 0"/>
+    <axis xyz="0 0 0"/>
     <dynamics damping="0.7"/>
   </joint>
@@ -194,7 +199,166 @@
     </collision>
     <visual>
-      <origin xyz="0.4 -0.4 0.05" rpy="0 3.14 0"/>
-      <geometry>
-	<mesh filename="package://arm_description/meshes/gearBox.STL" scale="0.2 0.2 0.2"/>
+      <origin xyz="${-elbow_width/5.5} ${-0.15-elbow_width/4.5} ${elbow_width/1.47}" rpy="0 3.14 0"/>
+      <geometry>
+	<mesh filename="package://arm_description/meshes/hand_assem.STL" scale="${scale} ${scale} ${scale}"/>
+      </geometry>
+      <material name="orange"/>
+    </visual>
+    <inertial>
+      <origin xyz="0 0 ${-elbow_width/2}" rpy="0 0 0"/>
+      <mass value="0.1"/>
+      <inertia
+	  ixx="0.1" ixy="0.0" ixz="0.0"
+	  iyy="0.1" iyz="0.0"
+	  izz="0.1"/>
+    </inertial>
+  </link>
+  <joint name="left_elbow1_1" type="continuous">
+    <parent link="link1"/>
+    <child link="left_elbow1"/>
+    <origin xyz="${x_offset} ${-width/2-leftArm_offset} ${height1-elbow_width/2}" rpy="0 0 3.14"/>
+    <axis xyz="0 1 0"/>
+    <dynamics damping="0.7"/>
+    <limit effort="${limit_effort}" lower="${limit_lower}" upper="${limit_upper}" velocity="${limit_velocity}" />
+    <safety_controller k_velocity="100" k_position="15" soft_lower_limit="-1.9" soft_upper_limit="0.5" />
+  </joint>
+  <link name="left_elbow1">
+    <collision>
+      <origin xyz="0 ${elbow_width/2} 0" rpy="0 0 0"/>
+      <geometry>
+	<box size="${elbow_width} ${elbow_width} ${elbow_width}"/>
+      </geometry>
+    </collision>
+    <visual>
+      <origin xyz="${-elbow_width/2} 0 ${-elbow_width/2}" rpy="0 0 0"/>
+      <geometry>
+	<mesh filename="package://arm_description/meshes/shoulder_ball.STL" scale="0.4 0.4 0.4"/>
+	<!--box size="${elbow_width} ${elbow_width} ${elbow_width}"/-->
+      </geometry>
+      <material name="orange"/>
+    </visual>
+    <inertial>
+      <origin xyz="0 ${elbow_width/2} 0" rpy="0 0 0"/>
+      <mass value="0.1"/>
+      <inertia
+	  ixx="0.1" ixy="0.0" ixz="0.0"
+	  iyy="0.1" iyz="0.0"
+	  izz="0.1"/>
+    </inertial>
+  </link>
+  <joint name="left_elbow1_2" type="continuous">
+    <parent link="left_elbow1"/>
+    <child link="left_link2"/>
+    <origin xyz="0 ${elbow_width/2+0.04} ${-elbow_width*0}" rpy="0 0 0"/>
+    <axis xyz="1 0 0"/>
+    <dynamics damping="0.7"/>
+  </joint>
+  <!-- Middle Link -->
+  <link name="left_link2">
+    <collision>
+      <origin xyz="0 0 ${-height2/2}" rpy="0 0 0"/>
+      <geometry>
+	<box size="${width} ${width} ${height2}"/>
+      </geometry>
+    </collision>
+    <visual>
+      <origin xyz="${-elbow_width/2.7} ${-y_offset-0.4} ${height2/3.5}" rpy="-1.57 0 0"/>
+      <geometry>
+	<mesh filename="package://arm_description/meshes/shoulder_link.STL" scale="0.4 0.4 0.4"/>
+      </geometry>
+      <material name="orange"/>
+    </visual>
+    <inertial>
+      <origin xyz="0 0 ${-height2/2}" rpy="0 0 0"/>
+      <mass value="0.1"/>
+      <inertia
+	  ixx="10.1" ixy="0.0" ixz="0.0"
+	  iyy="10.1" iyz="0.0"
+	  izz="10.1"/>
+    </inertial>
+  </link>
+  <joint name="left_elbow2_1" type="continuous">
+    <parent link="left_link2"/>
+    <child link="left_elbow2"/>
+    <origin xyz="0 0 ${-height2-z_offset}" rpy="0 0 0"/>
+    <axis xyz="0 0 1"/>
+    <dynamics damping="0.7"/>
+    <limit effort="${limit_effort}" lower="${limit_lower}" upper="${limit_upper}" velocity="${limit_velocity}" />
+    <safety_controller k_velocity="100" k_position="15" soft_lower_limit="-1.9" soft_upper_limit="0.5" />
+  </joint>
+  <!-- Elbow 2 Link -->
+  <link name="left_elbow2">
+    <collision>
+      <origin xyz="0 0 ${-elbow_width/2}" rpy="0 0 0"/>
+      <geometry>
+	<box size="${elbow_width} ${elbow_width} ${elbow_width}"/>
+      </geometry>
+    </collision>
+    <visual>
+      <origin xyz="${-elbow_width/2.5} ${-elbow_width/4-y_offset} ${z_offset-0.08}" rpy="-1.57 0 0"/>
+      <geometry>
+	<mesh filename="package://arm_description/meshes/elbow_ball.STL" scale="${scale} ${scale} ${scale}"/>
+      </geometry>
+      <material name="orange"/>
+    </visual>
+    <inertial>
+      <origin xyz="0 0 ${-elbow_width/2}" rpy="0 0 0"/>
+      <mass value="0.1"/>
+      <inertia
+	  ixx="0.1" ixy="0.0" ixz="0.0"
+	  iyy="0.1" iyz="0.0"
+	  izz="0.1"/>
+    </inertial>
+  </link>
+  <joint name="left_elbow2_2" type="continuous">
+    <parent link="left_elbow2"/>
+    <child link="left_link3"/>
+    <origin xyz="0 0 ${-elbow_width/2}" rpy="0 0 0"/>
+    <axis xyz="1 0 0"/>
+    <dynamics damping="0.7"/>
+  </joint>
+  <!-- Forearm Link -->
+  <link name="left_link3">
+    <collision>
+      <origin xyz="0 0 ${-height3/2}" rpy="0 0 0"/>
+      <geometry>
+	<box size="${width} ${width} ${height3}"/>
+      </geometry>
+    </collision>
+    <visual>
+      <origin xyz="${-elbow_width/4.1} ${-elbow_width/4-y_offset} ${z_offset+0.3}" rpy="-1.57 0 0"/>
+      <geometry>
+	<mesh filename="package://arm_description/meshes/forearm_link.STL" scale="${scale} ${scale} ${scale}"/>
+      </geometry>
+      <material name="black"/>
+    </visual>
+    <inertial>
+      <origin xyz="0 0 ${-height3/2}" rpy="0 0 0"/>
+      <mass value="0.1"/>
+      <inertia
+	  ixx="3.1" ixy="0.0" ixz="0.0"
+	  iyy="3.1" iyz="0.0"
+	  izz="3.1"/>
+    </inertial>
+  </link>
+  <joint name="left_elbow3_1" type="continuous">
+    <parent link="left_link3"/>
+    <child link="left_elbow3"/>
+    <origin xyz="0 ${0.15-y_offset} ${-1.79+z_offset}" rpy="0 0 0"/>
+    <axis xyz="0 0 0"/>
+    <dynamics damping="0.7"/>
+  </joint>
+  <!-- Hand Link -->
+  <link name="left_elbow3">
+    <collision>
+      <origin xyz="0 0 ${-elbow_width/2}" rpy="0 0 0"/>
+      <geometry>
+	<box size="${elbow_width} ${elbow_width} ${elbow_width}"/>
+      </geometry>
+    </collision>
+    <visual>
+      <origin xyz="${elbow_width/3.5} ${-elbow_width/2.7} ${-elbow_width/1.37}" rpy="0 0 0"/>
+      <geometry>
+	<mesh filename="package://arm_description/meshes/hand_assem_left.STL" scale="${scale} ${scale} ${scale}"/>
       </geometry>
       <material name="orange"/>
@@ -259,3 +423,53 @@
     </actuator>
   </transmission>
+ <transmission name="left_tran_elbow1_1">
+    <type>transmission_interface/SimpleTransmission</type>
+    <joint name="left_elbow1_1">
+      <hardwareInterface>EffortJointInterface</hardwareInterface>
+    </joint>
+    <actuator name="left_motor1_1">
+      <hardwareInterface>EffortJointInterface</hardwareInterface>
+      <mechanicalReduction>1</mechanicalReduction>
+    </actuator>
+  </transmission>
+  <transmission name="left_tran_elbow1_2">
+    <type>transmission_interface/SimpleTransmission</type>
+    <joint name="left_elbow1_2">
+      <hardwareInterface>EffortJointInterface</hardwareInterface>
+    </joint>
+    <actuator name="left_motor1_2">
+      <hardwareInterface>EffortJointInterface</hardwareInterface>
+      <mechanicalReduction>1</mechanicalReduction>
+    </actuator>
+  </transmission>
+  <transmission name="left_tran_elbow2_1">
+    <type>transmission_interface/SimpleTransmission</type>
+    <joint name="left_elbow2_1">
+      <hardwareInterface>EffortJointInterface</hardwareInterface>
+    </joint>
+    <actuator name="left_motor2_1">
+      <hardwareInterface>EffortJointInterface</hardwareInterface>
+      <mechanicalReduction>1</mechanicalReduction>
+    </actuator>
+  </transmission>
+  <transmission name="left_tran_elbow2_2">
+    <type>transmission_interface/SimpleTransmission</type>
+    <joint name="left_elbow2_2">
+      <hardwareInterface>EffortJointInterface</hardwareInterface>
+    </joint>
+    <actuator name="left_motor2_2">
+      <hardwareInterface>EffortJointInterface</hardwareInterface>
+      <mechanicalReduction>1</mechanicalReduction>
+    </actuator>
+  </transmission>
+  <transmission name="left_tran_elbow3_1">
+    <type>transmission_interface/SimpleTransmission</type>
+    <joint name="left_elbow3_1">
+      <hardwareInterface>EffortJointInterface</hardwareInterface>
+    </joint>
+    <actuator name="left_motor3_1">
+      <hardwareInterface>EffortJointInterface</hardwareInterface>
+      <mechanicalReduction>1</mechanicalReduction>
+    </actuator>
+  </transmission>
 </robot>
